Commit message: Swimming Pool Done

File: uuv_descriptions/world_models/bucket3.SLDPRT/urdf/bucket3.SLDPRT.urdf (robot description, URDF)
Before this commit: robot bucket2.SLDPRT, 1 links, 0 joints
Links:
- removed link bucket2.SLDPRT
- added link bucket3.SLDPRT, mass 1.53; collision mesh filename=package://bucket3.SLDPRT/meshes/bucket3.SLDPRT.STL; visual mesh filename=package://bucket3.SLDPRT/meshes/bucket3.SLDPRT.STL

File: uuv_descriptions/world_models/pole-pinger.SLDPRT/urdf/pole-pinger.SLDPRT.urdf (robot description, URDF)
Before this commit: robot pole-pinger.SLDPRT, 1 links, 0 joints
Links:
- link pole-pinger.SLDPRT: mass 9.4154 -> 9.4074
