Commit message: Added models without color

File: niot_description/models/niot_candy/urdf/niot_candy.urdf (robot description, URDF)
Before this commit: robot niot_path, 1 links, 0 joints
Links:
- link base_link: mass 2.5722 -> 0.55615; geometry collision mesh filename=package://niot_candy/meshes/base_link.STL; visual mesh filename=package://niot_candy/meshes/base_link.STL

File: niot_description/models/niot_flower_green/urdf/niot_flower_green.urdf (robot description, URDF)
Before this commit: robot niot_path, 1 links, 0 joints
Links:
- link base_link: mass 2.5722 -> 7.2406; geometry collision mesh filename=package://niot_flower_green/meshes/base_link.STL; visual mesh filename=package://niot_flower_green/meshes/base_link.STL

File: niot_description/models/niot_flower_red/urdf/niot_flower_red.urdf (robot description, URDF)
Before this commit: robot niot_path, 1 links, 0 joints
Links:
- link base_link: mass 2.5722 -> 7.5827; geometry collision mesh filename=package://niot_flower_red/meshes/base_link.STL; visual mesh filename=package://niot_flower_red/meshes/base_link.STL

File: niot_description/models/niot_flower_yellow/urdf/niot_flower_yellow.urdf (robot description, URDF)
Before this commit: robot niot_path, 1 links, 0 joints
Links:
- link base_link: mass 2.5722 -> 7.3927; geometry collision mesh filename=niot_flower_yellow/meshes/base_link.STL; visual mesh filename=package://niot_flower_yellow/meshes/base_link.STL

File: niot_description/models/niot_gate/urdf/niot_gate.urdf (robot description, URDF)
Before this commit: robot niot_path, 1 links, 0 joints
Links:
- link base_link: mass 2.5722 -> 7.0204; geometry collision mesh filename=package://niot_gate/meshes/base_link.STL; visual mesh filename=package://niot_gate/meshes/base_link.STL

File: niot_description/models/niot_torpedo/urdf/niot_torpedo.urdf (robot description, URDF)
Before this commit: robot niot_path, 1 links, 0 joints
Links:
- link base_link: mass 2.5722 -> 11.226; geometry collision mesh filename=package://niot_torpedo/meshes/base_link.STL; visual mesh filename=package://niot_torpedo/meshes/base_link.STL
