Commit message: Added somethings

File: niot_description/models/anahita/urdf/anahita.urdf (robot description, URDF)
Before this commit: robot anahita, 12 links, 10 joints
Joints:
- added joint east_joint: type fixed, parent base_link, child east, origin xyz=-0.00295011291907577 0.0748526601695768 -0.30691889078886 rpy=-6.12319392837392E-17 0.00727776166092887 -4.45627526281709E-19, axis 0 0 0

File: niot_description/models/niot_flower_red/urdf/niot_flower_red.urdf (robot description, URDF)
Before this commit: robot niot_flower_red, 1 links, 0 joints
Links:
- link base_link: geometry collision mesh filename=package://niot_flower_red/meshes/base_link.STL scale=0.75 0.75 0.75; visual mesh filename=package://niot_flower_red/meshes/base_link.STL scale=0.75 0.75 0.75
